File: ZYNQ_PMU.kicad_sch (KiCad schematic)
At the start: 0 parts

Commit message: Update JTAG and SDR schematics and libraries
Parts:
- added U10, U11, U12, U13, U9: MP2145GD-Z, easyeda2kicad:QFN-12_L3.0-W2.0_MP2145GD-Z, symbol ZYNQ7020_SDR:MP2145GD-Z
- added U14: TPS51200DRCR, easyeda2kicad:WSON-10_L3.0-W3.0-P0.50-BL-EP, symbol ZYNQ7020_SDR:TPS51200DRCR
