File: ZYNQ_USB_PHY.kicad_sch (KiCad schematic)
At the start: 0 parts

Commit message: Update JTAG and SDR schematics and libraries
Parts:
- added U4: USB3320C-EZK-TR, easyeda2kicad:QFN-32_L5.0-W5.0-P0.50-BL-EP3.4, symbol ZYNQ7020_SDR:USB3320C-EZK-TR
Changed lines of the file:
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@@
 	(generator_version "10.0")
 	(paper "A4")
+	(symbol
+		(lib_id "ZYNQ7020_SDR:USB3320C-EZK-TR")
+		(at 129.54 95.25 0)
+		(unit 1)
+		(body_style 1)
+		(exclude_from_sim no)
+		(in_bom yes)
+		(on_board yes)
+		(in_pos_files yes)
+		(dnp no)
+		(fields_autoplaced yes)
+		(property "Reference" "U4"
+			(at 140.5733 71.12 0)
+			(show_name no)
+			(do_not_autoplace no)
+			(effects
+				(font
+					(size 1.27 1.27)
+				)
+				(justify left)
+			)
+		)
+		(property "Value" "USB3320C-EZK-TR"
+			(at 140.5733 73.66 0)
+			(show_name no)
+			(do_not_autoplace no)
+			(effects
+				(font
+					(size 1.27 1.27)
+				)
+				(justify left)
+			)
+		)
+		(property "Footprint" "easyeda2kicad:QFN-32_L5.0-W5.0-P0.50-BL-EP3.4"
+			(at 129.54 124.46 0)
+			(hide yes)
+			(show_name no)
+			(do_not_autoplace no)
+			(effects
+				(font
+					(size 1.27 1.27)
+				)
+			)
+		)
+		(property "Datasheet" "https://lcsc.com/product-detail/USB_MICROCHIP_USB3320C-EZK-TR_USB3320C-EZK-TR_C132156.html"
+			(at 129.54 127 0)
+			(hide yes)
+			(show_name no)
+			(do_not_autoplace no)
+			(effects
+				(font
+					(size 1.27 1.27)
+				)
+			)
+		)
+		(property "Description" ""
+			(at 129.54 95.25 0)
+			(hide yes)
+			(show_name no)
+			(do_not_autoplace no)
+			(effects
+				(font
+					(size 1.27 1.27)
+				)
+			)
+		)
+		(property "Manufacturer" "MICROCHIP(美国微芯)"
+			(at 129.54 129.54 0)
+			(hide yes)
+			(show_name no)
+			(do_not_autoplace no)
+			(effects
+				(font
+					(size 1.27 1.27)
+				)
+			)
+		)
+		(property "MPN" "USB3320C-EZK-TR"
+			(at 129.54 132.08 0)
+			(hide yes)
+			(show_name no)
+			(do_not_autoplace no)
+			(effects
+				(font
+					(size 1.27 1.27)
+				)
+			)
+		)
+		(property "LCSC Part" "C132156"
+			(at 129.54 134.62 0)
+			(hide yes)
+			(show_name no)
+			(do_not_autoplace no)
+			(effects
+				(font
+					(size 1.27 1.27)
+				)
+			)
+		)
+		(pin "1"
+		)
+		(pin "6"
+		)
+		(pin "4"
+		)
+		(pin "3"
+		)
+		(pin "2"
+		)
+		(pin "5"
+		)
+		(pin "33"
+		)
+		(pin "32"
+		)
+		(pin "24"
+		)
+		(pin "19"
+		)
+		(pin "17"
+		)
+		(pin "7"
+		)
+		(pin "27"
+		)
+		(pin "8"
+		)
+		(pin "23"
+		)
+		(pin "20"
+		)
+		(pin "26"
+		)
+		(pin "30"
+		)
+		(pin "22"
+		)
+		(pin "31"
+		)
+		(pin "12"
+		)
+		(pin "21"
+		)
+		(pin "9"
+		)
+		(pin "28"
+		)
+		(pin "29"
+		)
+		(pin "16"
+		)
+		(pin "18"
+		)
+		(pin "13"
+		)
+		(pin "15"
+		)
+		(pin "14"
+		)
+		(pin "25"
+		)
+		(pin "10"
+		)
+		(pin "11"
+		)
+		(instances
+			(project "ZYNQ7020_SDR"
+				(path "/3a68e3c4-732f-4f36-849e-450e7f6f5412/f9fafe9c-4ce3-4d73-be49-33280a5ea425"
+					(reference "U4")
+					(unit 1)
+				)
+			)
+		)
+	)
 )
